Commit message: allegro hand now appears in paused simulation

File: ros_packages/src/allegro_right_hand_description/model/allegro_hand_description_right.xacro (robot description, xacro)
@@ -37,5 +37,5 @@
   <xacro:property name="limit_2_low" 					value="-0.274"/>
   <xacro:property name="limit_3_up" 					value="1.718"/>
-  <xacro:property name="limit_3_low" 					value=" -0.327"/>
+  <xacro:property name="limit_3_low" 					value="-0.327"/>
   <xacro:property name="limit_0_t_up"  				value="1.496"/>
   <xacro:property name="limit_0_t_low" 				value="0.363"/>
@@ -56,7 +56,4 @@
       </geometry>
       <origin rpy="0 0 0" xyz="0 0 0 "/>
-      <material name="black">
-        <color rgba="0.2 0.2 0.2 1"/>
-      </material>
     </visual>
     <collision>
@@ -66,4 +63,5 @@
         <!-- <mesh filename="package://allegro_right_hand_description/model/meshes/base_link.STL"/> -->
       </geometry>
+      <origin rpy="0 0 0" xyz="-0.009300 0 -${palm_link_z/2}"/>
     </collision>
     <inertial>
@@ -87,7 +85,4 @@
           <mesh filename="package://allegro_right_hand_description/model/meshes/link_12.0_right.STL"/>
         </geometry>
-        <material name="black">
-          <color rgba=".2 .2 .2 1"/>
-        </material>
         <!-- <origin rpy="${180*DEG2RAD} 0 0" xyz="0 0 0"/> -->
       </visual>
@@ -97,5 +92,5 @@
           <mesh filename="package://allegro_right_hand_description/model/meshes/link_12.0_right.STL"/>
         </geometry>
-        <!-- <origin rpy="0 0 0" xyz="${-0.0358/2+0.0} ${.018/2} ${.029/2}"/> -->
+        <origin rpy="0 0 0" xyz="${-0.0358/2+0.0} ${.018/2} ${.029/2}"/>
       </collision>
       <inertial>
@@ -109,5 +104,4 @@
     	<origin rpy="${finger_angle_r} ${finger_angle_p} ${finger_angle_y}"
               xyz="${offset_origin_x} ${offset_origin_y} ${offset_origin_z}"/>
-      <!-- <origin xyz="0.1 0 0" rpy="0 0 0"/> -->
       <axis xyz="-1 0 0"/>
       <limit effort="15" velocity="7"
@@ -124,7 +118,4 @@
           <mesh filename="package://allegro_right_hand_description/model/meshes/link_13.0.STL"/>
         </geometry>
-        <material name="black">
-          <color rgba=".2 .2 .2 1"/>
-        </material>
       </visual>
       <collision>
@@ -133,5 +124,5 @@
           <mesh filename="package://allegro_right_hand_description/model/meshes/link_13.0.STL"/>
         </geometry>
-        <!-- <origin rpy="0 0 0" xyz="0 0 ${link1_t_z/2}"/> -->
+        <origin rpy="0 0 0" xyz="0 0 ${link1_t_z/2}"/>
       </collision>
       <inertial>
@@ -158,6 +149,4 @@
           <mesh filename="package://allegro_right_hand_description/model/meshes/link_14.0.STL"/>
         </geometry>
-        <material name="black">
-        </material>
       </visual>
       <collision>
@@ -166,5 +155,5 @@
           <mesh filename="package://allegro_right_hand_description/model/meshes/link_14.0.STL"/>
         </geometry>
-        <!-- <origin rpy="0 0 0" xyz="0 0 ${link2_t_z/2}"/> -->
+        <origin rpy="0 0 0" xyz="0 0 ${link2_t_z/2}"/>
       </collision>
       <inertial>
@@ -197,5 +186,5 @@
           <mesh filename="package://allegro_right_hand_description/model/meshes/link_15.0.STL"/>
         </geometry>
-        <!-- <origin rpy="0 0 0" xyz="0 0 ${(link3_t_z-fingerTip_r)/2}"/> -->
+        <origin rpy="0 0 0" xyz="0 0 ${(link3_t_z-fingerTip_r)/2}"/>
       </collision>
       <inertial>
@@ -223,7 +212,4 @@
           <mesh filename="package://allegro_right_hand_description/model/meshes/link_15.0_tip.STL"/>
         </geometry>
-        <material name="white">
-          <color rgba=".9 .9 .9 1"/>
-        </material>
       </visual>
       <collision>
@@ -232,5 +218,5 @@
           <mesh filename="package://allegro_right_hand_description/model/meshes/link_15.0_tip.STL"/>
         </geometry>
-        <!-- <origin rpy="0 0 0" xyz="0 0 0"/> -->
+        <origin rpy="0 0 0" xyz="0 0 0"/>
       </collision>
       <inertial>
@@ -256,5 +242,4 @@
           <mesh filename="package://allegro_right_hand_description/model/meshes/link_0.0.STL"/>
         </geometry>
-        <material name="black"/>
       </visual>
       <collision>
@@ -270,4 +255,5 @@
       </inertial>
     </link>
+    <gazebo reference="link_${finger_num*4+0}"><material>Gazebo/Blue</material></gazebo>
     <joint name="joint_${finger_num*4+0}" type="revolute">
       <axis xyz="0 0 1"/>
@@ -287,5 +273,4 @@
           <mesh filename="package://allegro_right_hand_description/model/meshes/link_1.0.STL"/>
         </geometry>
-        <material name="black"/>
       </visual>
       <collision>
@@ -301,4 +286,5 @@
       </inertial>
     </link>
+    <gazebo reference="link_${finger_num*4+1}"><material>Gazebo/Black</material></gazebo>
     <joint name="joint_${finger_num*4+1}" type="revolute">
       <limit effort="15" velocity="7"
@@ -317,5 +303,4 @@
           <mesh filename="package://allegro_right_hand_description/model/meshes/link_2.0.STL"/>
         </geometry>
-        <material name="black"/>
       </visual>
       <collision>
@@ -331,4 +316,5 @@
       </inertial>
     </link>
+    <gazebo reference="link_${finger_num*4+2}"><material>Gazebo/Red</material></gazebo>
     <joint name="joint_${finger_num*4+2}" type="revolute">
       <axis xyz="0 1 0"/>
@@ -347,5 +333,4 @@
           <mesh filename="package://allegro_right_hand_description/model/meshes/link_3.0.STL"/>
         </geometry>
-        <material name="black"/>
       </visual>
       <collision>
@@ -361,4 +346,5 @@
       </inertial>
     </link>
+    <gazebo reference="link_${finger_num*4+3}"><material>Gazebo/Orange</material></gazebo>
     <joint name="joint_${finger_num*4+3}" type="revolute">
       <axis xyz="0 1 0"/>
@@ -377,7 +363,4 @@
           <mesh filename="package://allegro_right_hand_description/model/meshes/link_3.0_tip.STL"/>
         </geometry>
-        <material name="white">
-          <color rgba=".9 .9 .9 1"/>
-        </material>
       </visual>
       <collision>
@@ -392,4 +375,5 @@
       </inertial>
     </link>
+    <gazebo reference="link_${finger_num*4+3}_tip"><material>Gazebo/White</material></gazebo>
     <joint name="joint_${finger_num*4+3}_tip" type="fixed">
       <parent link="link_${finger_num*4+3}"/>
@@ -403,5 +387,5 @@
   <!-- RIGHT HAND due to which finger is number 0 -->
   <!-- for LEFT HAND switch the sign of the **offset_origin_y** and **finger_angle_r** parameters-->
-  <!--<xacro:finger
+  <xacro:finger
           finger_num="0"
           offset_origin_x="${offset_origin_x_const}"
@@ -423,5 +407,5 @@
           offset_origin_z="${offset_origin_z_const}"
           finger_angle_r="${5.0*DEG2RAD}"
-          /> -->
+          />
   <!-- THUMB -->
   <xacro:thumb_right
