Commit message: added and tested allegro right hand direct geometric model

File: ros_packages/src/allegro_right_hand_description/model/allegro_right_hand_description.urdf.xacro (robot description, xacro)
@@ -5,20 +5,20 @@
   <gazebo>
     <plugin name="allegro_right_hand_control_plugin" filename="liballegro_right_hand_control_plugin.so">
-    	<index_joint1_init>0.40</index_joint1_init>
-    	<index_joint2_init>0.50</index_joint2_init>
-    	<index_joint3_init>0.70</index_joint3_init>
-    	<index_joint4_init>0.70</index_joint4_init>
-    	<middle_joint1_init>0.20</middle_joint1_init>
-    	<middle_joint2_init>0.20</middle_joint2_init>
-    	<middle_joint3_init>0.20</middle_joint3_init>
-    	<middle_joint4_init>0.20</middle_joint4_init>
-    	<pinky_joint1_init>0.30</pinky_joint1_init>
-    	<pinky_joint2_init>0.30</pinky_joint2_init>
-    	<pinky_joint3_init>0.30</pinky_joint3_init>
-    	<pinky_joint4_init>0.30</pinky_joint4_init>
-    	<thumb_joint1_init>0.70</thumb_joint1_init>
-    	<thumb_joint2_init>0.20</thumb_joint2_init>
-    	<thumb_joint3_init>0.70</thumb_joint3_init>
-    	<thumb_joint4_init>0.70</thumb_joint4_init>
+    	<index_joint1_init>0.00</index_joint1_init>
+    	<index_joint2_init>0.00</index_joint2_init>
+    	<index_joint3_init>0.00</index_joint3_init>
+    	<index_joint4_init>0.00</index_joint4_init>
+    	<middle_joint1_init>0.00</middle_joint1_init>
+    	<middle_joint2_init>0.00</middle_joint2_init>
+    	<middle_joint3_init>0.00</middle_joint3_init>
+    	<middle_joint4_init>0.00</middle_joint4_init>
+    	<pinky_joint1_init>0.00</pinky_joint1_init>
+    	<pinky_joint2_init>0.00</pinky_joint2_init>
+    	<pinky_joint3_init>0.00</pinky_joint3_init>
+    	<pinky_joint4_init>0.00</pinky_joint4_init>
+    	<thumb_joint1_init>-0.027</thumb_joint1_init>
+    	<thumb_joint2_init>0.00</thumb_joint2_init>
+    	<thumb_joint3_init>0.77</thumb_joint3_init>
+    	<thumb_joint4_init>0.77</thumb_joint4_init>
     </plugin>
   </gazebo>

File: ros_packages/src/allegro_right_hand_description/model/allegro_right_hand_description.xacro (robot description, xacro)
@@ -113,5 +113,6 @@
       <parent link="palm_link"/>
       <child link="${finger_name}_link0"/>s
-      <dynamics damping="3" friction="10"/>
+      <!-- <dynamics damping="3" friction="10"/> -->
+      <dynamics damping="1" friction="1"/>
     </joint>
     <!-- [LINK 13] -->
@@ -146,5 +147,6 @@
       <child link="${finger_name}_link1"/>
       <origin xyz="-0.027 0.005 0.0399"/>
-      <dynamics damping="3" friction="5"/>
+      <!-- <dynamics damping="3" friction="5"/> -->
+      <dynamics damping="1" friction="1"/>
     </joint>
     <!-- [LINK 14] -->
@@ -179,5 +181,6 @@
       <child link="${finger_name}_link2"/>
       <origin xyz="0 0 ${link1_t_z}"/>
-      <dynamics damping="3" friction="10"/>
+      <!-- <dynamics damping="3" friction="10"/> -->
+      <dynamics damping="1" friction="1"/>
     </joint>
     <!-- [LINK 15] -->
@@ -212,5 +215,6 @@
       <child link="${finger_name}_link3"/>
       <origin xyz="0 0 ${link2_t_z}"/>
-      <dynamics damping="3" friction="12"/>
+      <!-- <dynamics damping="3" friction="12"/> -->
+      <dynamics damping="1" friction="1"/>
     </joint>
     <!-- [FINGER TIP] -->

Commit message: allegro-right-hand individual finger position control is now working

File: ros_packages/src/allegro_right_hand_description/model/allegro_right_hand_description.urdf.xacro (robot description, xacro)
@@ -6,20 +6,36 @@
     <!-- <plugin name="allegro_right_hand_control_plugin" filename="liballegro_right_hand_control_plugin.so"> -->
     <plugin name="generic_interface_plugin" filename="libgeneric_interface_plugin.so">
-    	<index_joint1_init>0.00</index_joint1_init>
-    	<index_joint2_init>0.00</index_joint2_init>
-    	<index_joint3_init>0.00</index_joint3_init>
-    	<index_joint4_init>0.00</index_joint4_init>
+    	<!-- <index_joint1_init>0.00</index_joint1_init>
+    	<index_joint2_init>0.10</index_joint2_init>
+    	<index_joint3_init>0.10</index_joint3_init>
+    	<index_joint4_init>0.10</index_joint4_init>
     	<middle_joint1_init>0.00</middle_joint1_init>
-    	<middle_joint2_init>0.00</middle_joint2_init>
-    	<middle_joint3_init>0.00</middle_joint3_init>
-    	<middle_joint4_init>0.00</middle_joint4_init>
+    	<middle_joint2_init>0.10</middle_joint2_init>
+    	<middle_joint3_init>0.10</middle_joint3_init>
+    	<middle_joint4_init>0.10</middle_joint4_init>
     	<pinky_joint1_init>0.00</pinky_joint1_init>
-    	<pinky_joint2_init>0.00</pinky_joint2_init>
-    	<pinky_joint3_init>0.00</pinky_joint3_init>
-    	<pinky_joint4_init>0.00</pinky_joint4_init>
-    	<thumb_joint1_init>-0.027</thumb_joint1_init>
-    	<thumb_joint2_init>0.00</thumb_joint2_init>
-    	<thumb_joint3_init>0.77</thumb_joint3_init>
-    	<thumb_joint4_init>0.77</thumb_joint4_init>
+    	<pinky_joint2_init>0.10</pinky_joint2_init>
+    	<pinky_joint3_init>0.10</pinky_joint3_init>
+    	<pinky_joint4_init>0.10</pinky_joint4_init>
+    	<thumb_joint1_init>0.5</thumb_joint1_init>
+    	<thumb_joint2_init>0.10</thumb_joint2_init>
+    	<thumb_joint3_init>0.10</thumb_joint3_init>
+    	<thumb_joint4_init>0.10</thumb_joint4_init> -->
+    	<joint1_init>0.000</joint1_init>
+    	<joint2_init>0.500</joint2_init>
+    	<joint3_init>0.500</joint3_init>
+    	<joint4_init>0.500</joint4_init>
+    	<joint5_init>0.000</joint5_init>
+    	<joint6_init>0.100</joint6_init>
+    	<joint7_init>0.100</joint7_init>
+    	<joint8_init>0.100</joint8_init>
+    	<joint9_init>0.000</joint9_init>
+    	<joint10_init>0.10</joint10_init>
+    	<joint11_init>0.10</joint11_init>
+    	<joint12_init>0.10</joint12_init>
+    	<joint13_init>0.50</joint13_init>
+    	<joint14_init>0.30</joint14_init>
+    	<joint15_init>0.30</joint15_init>
+    	<joint16_init>0.30</joint16_init>
     </plugin>
   </gazebo>

File: ros_packages/src/allegro_right_hand_description/model/allegro_right_hand_description.xacro (robot description, xacro)
@@ -46,4 +46,21 @@
   <xacro:property name="limit_3_t_up"  				value="1.819"/>
   <xacro:property name="limit_3_t_low" 				value="-0.262"/>
+  <!-- <xacro:property name="joint_safety_margin" 	value="0.0"/>
+  <xacro:property name="limit_0_up" 					value="0.0"/>
+  <xacro:property name="limit_0_low" 					value="-0.0"/>
+  <xacro:property name="limit_1_up" 					value="0.0"/>
+  <xacro:property name="limit_1_low" 					value="-0.0"/>
+  <xacro:property name="limit_2_up" 					value="0.0"/>
+  <xacro:property name="limit_2_low" 					value="-0.0"/>
+  <xacro:property name="limit_3_up" 					value="0.0"/>
+  <xacro:property name="limit_3_low" 					value="-0.0"/>
+  <xacro:property name="limit_0_t_up"  				value="0.0"/>
+  <xacro:property name="limit_0_t_low" 				value="0.0"/>
+  <xacro:property name="limit_1_t_up"  				value="0.0"/>
+  <xacro:property name="limit_1_t_low" 				value="-0.0"/>
+  <xacro:property name="limit_2_t_up"  				value="0.0"/>
+  <xacro:property name="limit_2_t_low" 				value="-0.0"/>
+  <xacro:property name="limit_3_t_up"  				value="0.0"/>
+  <xacro:property name="limit_3_t_low" 				value="-0.0"/> -->
   <!-- ============================================================================= -->
   <!-- Base link -->
