Commit message: refactoring#2

File: ros_packages/src/allegro_right_hand_description/model/allegro_right_hand.urdf.xacro (robot description, xacro)
@@ -1,6 +1,19 @@
 <?xml version='1.0' encoding='utf-8'?>
 <robot xmlns:xacro="http://www.ros.org/wiki/xacro" name="allegro_right_hand_description">
+  <xacro:property name="robot_arm1" value="panda1" />
+  <!-- Franka-Panda arm to Allegro hand connection -->
+  <xacro:include filename="$(find urdf_models)/models/panda_allegro_connection/panda_allegro_connection.xacro"/>
+  <xacro:panda_allegro_connection connected_to="" ns="${robot_arm1}" xyz="0 0 0.107" rpy="0 0 0" />
+  <!-- Allegro right hand model -->
+  <xacro:include filename="$(find allegro_right_hand_description)/model/allegro_right_hand.xacro"/>
+  <!-- 0.0091=(-0.0113+0.0204) : -0.0113 to put the allegro hand Palm frame at zero position then add 0.0.0204(40.8mm/2) to put the same frame at center of panda-allegro-connection  -->
+  <xacro:allegro_right_hand ns="${robot_arm1}" x="-0.0091" y="0" z="0.02" roll="0" pitch="0" yaw="${pi}" connected_to="${robot_arm1}_panda_allegro_connection" />
+  <!-- ReadSense-d435 depth camera -->
+  <xacro:include filename="$(find realsense_d435_description)/model/realsense_d435.xacro"/>
+  <xacro:realsense_d435 connected_to="${robot_arm1}_panda_allegro_connection" ns="${robot_arm1}" origin_rpy="0 ${-pi/2} 0" origin_xyz="-0.0673 0 -0.02" />
+  <!--
   <xacro:include filename="$(find allegro_right_hand_description)/model/allegro_right_hand.xacro" />
   <xacro:allegro_right_hand ns="allegro_right_hand" roll="0" pitch="0" yaw="0" x="0" y="0" z="0" />
+   -->
   <!-- attach the custom make gazebo plugin "allegro_right_hand_control_plugin" -->
   <gazebo>

File: ros_packages/src/franka_panda_gripper_description/model/panda_gripper_gazebo.urdf.xacro (robot description, xacro)
@@ -3,5 +3,17 @@
   <!-- for .dae files visualization problem in Gazebo8 -->
   <transparent opaque="RGB_ZERO"> <color>1 1 1 1</color> </transparent> <transparency><float>1</float></transparency>
+  <xacro:property name="robot_arm1" value="panda1" />
+  <!-- Franka-Panda arm to Allegro hand connection -->
+  <xacro:include filename="$(find urdf_models)/models/panda_allegro_connection/panda_allegro_connection.xacro"/>
+  <xacro:panda_allegro_connection connected_to="" ns="${robot_arm1}" xyz="0 0 0.107" rpy="0 0 0" />
+  <!-- Allegro right hand model -->
+  <xacro:include filename="$(find franka_panda_gripper_description)/model/panda_gripper_gazebo.xacro"/>
+  <xacro:panda_gripper ns="${robot_arm1}" xyz="0 0 0.02" connected_to="${robot_arm1}_panda_allegro_connection" />
+  <!-- ReadSense-d435 depth camera -->
+  <xacro:include filename="$(find realsense_d435_description)/model/realsense_d435.xacro"/>
+  <xacro:realsense_d435 connected_to="${robot_arm1}_panda_allegro_connection" ns="${robot_arm1}" origin_rpy="0 ${-pi/2} 0" origin_xyz="-0.0673 0 -0.02" />
+  <!--
   <xacro:include filename="$(find franka_panda_gripper_description)/model/panda_gripper_gazebo.xacro"/>
   <xacro:panda_gripper ns="panda_arm" xyz="0 0 0.1" />
+   -->
 </robot>

File: ros_packages/src/franka_panda_gripper_description/model/panda_gripper_gazebo.xacro (robot description, xacro)
@@ -23,5 +23,5 @@
 	<visual>
 	<geometry>
-	<mesh filename="package://${description_pkg}/model/meshes/visual/hand.dae"/>
+	<mesh filename="package://${description_pkg}/model/meshes/visual/hand.stl"/>
 	</geometry>
 	</visual>
@@ -37,8 +37,10 @@
 	</inertial>
 </link>
+<gazebo reference="${ns}_hand"><material>Gazebo/Orange</material></gazebo>
 <link name="${ns}_leftfinger">
 	<visual>
+	<origin xyz="0 0.04 0" rpy="0 0 0"/>
 	<geometry>
-	<mesh filename="package://${description_pkg}/model/meshes/visual/finger.dae"/>
+	<mesh filename="package://${description_pkg}/model/meshes/visual/finger.stl"/>
 	</geometry>
 	</visual>
@@ -54,9 +56,10 @@
 	</inertial>
 </link>
+<gazebo reference="${ns}_leftfinger"><material>Gazebo/Red</material></gazebo>
 <link name="${ns}_rightfinger">
 	<visual>
-	<origin xyz="0 0 0" rpy="0 0 ${pi}"/>
+	<origin xyz="0 -0.04 0" rpy="0 0 ${pi}"/>
 	<geometry>
-	<mesh filename="package://${description_pkg}/model/meshes/visual/finger.dae"/>
+	<mesh filename="package://${description_pkg}/model/meshes/visual/finger.stl"/>
 	</geometry>
 	</visual>
@@ -73,4 +76,5 @@
 	</inertial>
 </link>
+<gazebo reference="${ns}_rightfinger"><material>Gazebo/Red</material></gazebo>
 <joint name="${ns}_finger_joint1" type="prismatic">
 	<parent link="${ns}_hand"/>

File: ros_packages/src/realsense_d435_description/model/realsense_d435.xacro (robot description, xacro)
@@ -87,4 +87,5 @@
     </collision>
   </link>
+  <gazebo reference="${ns}_link"><material>Gazebo/BlueGlow</material></gazebo>
   <!-- Virtual links representing the cameras positons and orientations-->
   <link name="${ns}_color" />

File: ros_packages/src/urdf_models/models/panda_allegro_connection/panda_allegro_connection.xacro (robot description, xacro)
@@ -38,5 +38,6 @@
   </inertial>
 </link>
-<gazebo reference="${ns}_panda_allegro_connection"><material>Gazebo/BlueGlow</material></gazebo>
+<!-- <gazebo reference="${ns}_panda_allegro_connection"><material>Gazebo/BlueGlow</material></gazebo> -->
+<gazebo reference="${ns}_panda_allegro_connection"><material>Gazebo/Green</material></gazebo>
 </xacro:macro>
 </robot>
