Commit message: code refinement#1

File: ros_packages/src/franka_panda_arm_plus_own_gripper_control_gazebo/model/panda_arm_plus_own_gripper_control_gazebo_plugin.urdf.xacro (robot description, xacro)
@@ -11,7 +11,7 @@
     <plugin name="franka_panda_arm_plus_own_gripper_control_plugin" filename="libfranka_panda_arm_plus_own_gripper_control_plugin.so">
     	<arm_joint1_init>0.00</arm_joint1_init>
-    	<arm_joint2_init>0.70</arm_joint2_init>
+    	<arm_joint2_init>-1.57</arm_joint2_init>
     	<arm_joint3_init>0.00</arm_joint3_init>
-    	<arm_joint4_init>0.00</arm_joint4_init>
+    	<arm_joint4_init>-1.57</arm_joint4_init>
     	<arm_joint5_init>0.00</arm_joint5_init>
     	<arm_joint6_init>0.00</arm_joint6_init>

File: ros_packages/src/franka_panda_control_gazebo/model/franka_panda_control_gazebo_plugin.urdf.xacro (robot description, xacro)
@@ -2,9 +2,10 @@
 <robot xmlns:xacro="http://www.ros.org/wiki/xacro" name="panda_arm">
   <xacro:include filename="$(find franka_panda_arm_description)/model/panda_arm_gazebo.xacro" />
-  <xacro:panda_arm arm_id="panda_arm" xyz="0 0 0" rpy="0 0 0" />
+  <xacro:panda_arm arm_id="panda_arm_1" xyz="0 0 0" rpy="0 0 0" />
   <!-- <xacro:panda_arm xyz="0 0 0.1" rpy="0 0 ${-pi/2}" /> -->
   <!-- attach the custom make gazebo plugin "franka_panda_control_plugin" -->
   <gazebo>
-    <plugin name="franka_panda_control_plugin" filename="libfranka_panda_control_plugin.so">
+    <!-- <plugin name="franka_panda_control_plugin" filename="libfranka_panda_control_plugin.so"> -->
+    <plugin name="generic_interface_plugin" filename="libgeneric_interface_plugin.so">
     	<joint1_init>0.00</joint1_init>
     	<joint2_init>-1.57</joint2_init>
@@ -16,3 +17,6 @@
     </plugin>
   </gazebo>
+  <gazebo reference="panda_arm::panda_arm_joint1">
+    <!--<provide_feedback>true<provide_feedback>-->
+  </gazebo>
 </robot>

File: ros_packages/src/franka_panda_gripper_description/model/panda_gripper_gazebo.xacro (robot description, xacro)
@@ -2,5 +2,5 @@
 <robot xmlns:xacro="http://www.ros.org/wiki/xacro" name="panda_gripper">
 <!-- robot constants -->
-<xacro:property name="mass" value="1" /> <!-- arbitrary value for mass -->
+<xacro:property name="mass" value="0.5" /> <!-- arbitrary value for mass -->
 <xacro:macro name="panda_gripper" params=" description_pkg:='franka_panda_gripper_description' connected_to:='' ns:='' rpy:='0 0 0' xyz:='0 0 0' ">
 <xacro:unless value="${connected_to == ''}">
@@ -33,5 +33,5 @@
 	<inertial>
 		<origin xyz="0 0 ${1/2}" rpy="0 0 0"/>
-		<mass value="${mass}"/>
+		<mass value="0.7"/>
 		<inertia ixx="0.0" ixy="0.0" ixz="0.0" iyy="0.0" iyz="0.0" izz="0.0"/>
 	</inertial>
@@ -50,5 +50,5 @@
 	<inertial>
 		<origin xyz="0 0 ${1/2}" rpy="0 0 0"/>
-		<mass value="${mass}"/>
+		<mass value="0.3"/>
 		<inertia ixx="0.0" ixy="0.0" ixz="0.0" iyy="0.0" iyz="0.0" izz="0.0"/>
 	</inertial>
@@ -69,5 +69,5 @@
 	<inertial>
 		<origin xyz="0 0 ${1/2}" rpy="0 0 0"/>
-		<mass value="${mass}"/>
+		<mass value="0.3"/>
 		<inertia ixx="0.0" ixy="0.0" ixz="0.0" iyy="0.0" iyz="0.0" izz="0.0"/>
 	</inertial>
