Commit message: code reorganizing + generic gazebo plugin + starting velocity control instead of torque control

File: ros_packages/src/franka_panda_arm_description/model/panda_arm_gazebo.xacro (robot description, xacro)
@@ -58,4 +58,5 @@
 <!-- Joint 1 -->
 <joint name="${arm_id}_joint1" type="revolute">
+  <provide_feedback>1</provide_feedback>
 	<safety_controller k_position="100.0" k_velocity="40.0" soft_lower_limit="-2.8973" soft_upper_limit="2.8973"/>
 	<origin rpy="0 0 0" xyz="0 0 0.333"/>
@@ -87,4 +88,5 @@
 <!-- Joint 2 -->
 <joint name="${arm_id}_joint2" type="revolute">
+  <provide_feedback>1</provide_feedback>
 	<safety_controller k_position="100.0" k_velocity="40.0" soft_lower_limit="-1.7628" soft_upper_limit="1.7628"/>
 	<origin rpy="${-pi/2} 0 0" xyz="0 0 0"/>
@@ -116,4 +118,5 @@
 <!-- Joint 3 -->
 <joint name="${arm_id}_joint3" type="revolute">
+  <provide_feedback>1</provide_feedback>
 	<safety_controller k_position="100.0" k_velocity="40.0" soft_lower_limit="-2.8973" soft_upper_limit="2.8973"/>
 	<origin rpy="${pi/2} 0 0" xyz="0 -0.316 0"/>
@@ -145,4 +148,5 @@
 <!-- Joint 4 -->
 <joint name="${arm_id}_joint4" type="revolute">
+  <provide_feedback>1</provide_feedback>
 	<safety_controller k_position="100.0" k_velocity="40.0" soft_lower_limit="-3.0718" soft_upper_limit="0.0175"/>
 	<origin rpy="${pi/2} 0 0" xyz="0.0825 0 0"/>
@@ -174,4 +178,5 @@
 <!-- Joint 5 -->
 <joint name="${arm_id}_joint5" type="revolute">
+  <provide_feedback>1</provide_feedback>
 	<safety_controller k_position="100.0" k_velocity="40.0" soft_lower_limit="-2.8973" soft_upper_limit="2.8973"/>
 	<origin rpy="${-pi/2} 0 0" xyz="-0.0825 0.384 0"/>
@@ -203,4 +208,5 @@
 <!-- Joint 6 -->
 <joint name="${arm_id}_joint6" type="revolute">
+  <physics><provide_feedback>true</provide_feedback></physics>
 	<safety_controller k_position="100.0" k_velocity="40.0" soft_lower_limit="-0.0175" soft_upper_limit="3.7525"/>
 	<origin rpy="${pi/2} 0 0" xyz="0 0 0"/>
@@ -232,4 +238,5 @@
 <!-- Joint 7 -->
 <joint name="${arm_id}_joint7" type="revolute">
+  <physics><provide_feedback>true</provide_feedback></physics>
 	<safety_controller k_position="100.0" k_velocity="40.0" soft_lower_limit="-2.8973" soft_upper_limit="2.8973"/>
 	<origin rpy="${pi/2} 0 0" xyz="0.088 0 0"/>
@@ -250,74 +257,4 @@
 	<axis xyz="0 0 0"/>
 </joint>
-<transmission name="${arm_id}_trans1">
-  <type>transmission_interface/SimpleTransmission</type>
-  <joint name="${arm_id}_joint1">
-    <hardwareInterface>hardware_interface/EffortJointInterface</hardwareInterface>
-  </joint>
-  <actuator name="${arm_id}_motor1">
-    <hardwareInterface>hardware_interface/EffortJointInterface</hardwareInterface>
-    <mechanicalReduction>1</mechanicalReduction>
-  </actuator>
-</transmission>
-<transmission name="${arm_id}_trans2">
-  <type>transmission_interface/SimpleTransmission</type>
-  <joint name="${arm_id}_joint2">
-    <hardwareInterface>hardware_interface/EffortJointInterface</hardwareInterface>
-  </joint>
-  <actuator name="${arm_id}_motor2">
-    <hardwareInterface>hardware_interface/EffortJointInterface</hardwareInterface>
-    <mechanicalReduction>1</mechanicalReduction>
-  </actuator>
-</transmission>
-<transmission name="${arm_id}_trans3">
-  <type>transmission_interface/SimpleTransmission</type>
-  <joint name="${arm_id}_joint3">
-    <hardwareInterface>hardware_interface/EffortJointInterface</hardwareInterface>
-  </joint>
-  <actuator name="${arm_id}_motor3">
-    <hardwareInterface>hardware_interface/EffortJointInterface</hardwareInterface>
-    <mechanicalReduction>1</mechanicalReduction>
-  </actuator>
-</transmission>
-<transmission name="${arm_id}_trans4">
-  <type>transmission_interface/SimpleTransmission</type>
-  <joint name="${arm_id}_joint4">
-    <hardwareInterface>hardware_interface/EffortJointInterface</hardwareInterface>
-  </joint>
-  <actuator name="${arm_id}_motor4">
-    <hardwareInterface>hardware_interface/EffortJointInterface</hardwareInterface>
-    <mechanicalReduction>1</mechanicalReduction>
-  </actuator>
-</transmission>
-<transmission name="${arm_id}_trans5">
-  <type>transmission_interface/SimpleTransmission</type>
-  <joint name="${arm_id}_joint5">
-    <hardwareInterface>hardware_interface/EffortJointInterface</hardwareInterface>
-  </joint>
-  <actuator name="${arm_id}_motor5">
-    <hardwareInterface>hardware_interface/EffortJointInterface</hardwareInterface>
-    <mechanicalReduction>1</mechanicalReduction>
-  </actuator>
-</transmission>
-<transmission name="${arm_id}_trans6">
-  <type>transmission_interface/SimpleTransmission</type>
-  <joint name="${arm_id}_joint6">
-    <hardwareInterface>hardware_interface/EffortJointInterface</hardwareInterface>
-  </joint>
-  <actuator name="${arm_id}_motor6">
-    <hardwareInterface>hardware_interface/EffortJointInterface</hardwareInterface>
-    <mechanicalReduction>1</mechanicalReduction>
-  </actuator>
-</transmission>
-<transmission name="${arm_id}_trans7">
-  <type>transmission_interface/SimpleTransmission</type>
-  <joint name="${arm_id}_joint7">
-    <hardwareInterface>hardware_interface/EffortJointInterface</hardwareInterface>
-  </joint>
-  <actuator name="${arm_id}_motor7">
-    <hardwareInterface>hardware_interface/EffortJointInterface</hardwareInterface>
-    <mechanicalReduction>1</mechanicalReduction>
-  </actuator>
-</transmission>
 </xacro:macro>
 </robot>

File: ros_packages/src/franka_panda_arm_plus_own_gripper_control_gazebo/model/panda_arm_plus_own_gripper_control_gazebo_plugin.urdf.xacro (robot description, xacro)
@@ -8,5 +8,5 @@
   <xacro:panda_gripper ns="gripper" rpy="0 0 ${-pi/4}" connected_to="panda_arm_link8"/>
   <!-- attach the custom make gazebo plugin "franka_panda_control_plugin" -->
-  <gazebo>
+  <!-- <gazebo>
     <plugin name="franka_panda_arm_plus_own_gripper_control_plugin" filename="libfranka_panda_arm_plus_own_gripper_control_plugin.so">
     	<arm_joint1_init>0.00</arm_joint1_init>
@@ -20,4 +20,17 @@
     	<gripper_joint2_init>0.00</gripper_joint2_init>
     </plugin>
+  </gazebo> -->
+  <gazebo>
+    <plugin name="generic_interface_plugin" filename="libgeneric_interface_plugin.so">
+    	<joint1_init>0.00</joint1_init>
+    	<joint2_init>-1.57</joint2_init>
+    	<joint3_init>0.00</joint3_init>
+    	<joint4_init>-1.57</joint4_init>
+    	<joint5_init>0.00</joint5_init>
+    	<joint6_init>0.00</joint6_init>
+    	<joint7_init>0.70</joint7_init>
+    	<joint8_init>0.00</joint8_init>
+    	<joint9_init>0.00</joint9_init>
+    </plugin>
   </gazebo>
 </robot>

Commit message: realsense gazebo ros plugin is now working

File: ros_packages/src/franka_panda_arm_description/model/panda_arm_gazebo.xacro (robot description, xacro)
@@ -29,5 +29,5 @@
 	<collision>
 		<geometry>
-		<mesh filename="package://${description_pkg}/model/meshes/collision/link0.stl"/>
+		<mesh filename="package://${description_pkg}/model/meshes/visual/link0.dae"/>
 		</geometry>
 	</collision>

File: ros_packages/src/franka_panda_arm_plus_allegro_right_hand_control_gazebo/model/franka_panda_arm_plus_allegro_right_hand_control_gazebo_plugin.urdf.xacro (robot description, xacro)
@@ -4,4 +4,5 @@
   <xacro:include filename="$(find allegro_right_hand_description)/model/allegro_right_hand.xacro"/>
   <xacro:panda_arm arm_id="panda_arm" xyz="0.62 0.138 0.986" rpy="0 0 ${pi/2}" />
+  <transparent opaque="RGB_ZERO"> <color>1 1 1 1</color> </transparent> <transparency><float>1</float></transparency>
   <link name="franka_panda_arm_allegro_hand_connection">
     <visual>
@@ -56,5 +57,31 @@
     	<joint22_init>0.70 </joint22_init>
     	<joint23_init>0.30 </joint23_init>
+    	<joint1_velocity_limit>1.0 </joint1_velocity_limit>
+    	<joint2_velocity_limit>1.0 </joint2_velocity_limit>
+    	<joint3_velocity_limit>1.0 </joint3_velocity_limit>
+    	<joint4_velocity_limit>1.0 </joint4_velocity_limit>
+    	<joint5_velocity_limit>1.0 </joint5_velocity_limit>
+    	<joint6_velocity_limit>1.0 </joint6_velocity_limit>
+    	<joint7_velocity_limit>1.0 </joint7_velocity_limit>
+    	<joint8_velocity_limit>1.0 </joint8_velocity_limit>
+    	<joint9_velocity_limit>1.0 </joint9_velocity_limit>
+    	<joint10_velocity_limit>1.0 </joint10_velocity_limit>
+    	<joint11_velocity_limit>1.0 </joint11_velocity_limit>
+    	<joint12_velocity_limit>1.0 </joint12_velocity_limit>
+    	<joint13_velocity_limit>1.0 </joint13_velocity_limit>
+    	<joint14_velocity_limit>1.0 </joint14_velocity_limit>
+    	<joint15_velocity_limit>1.0 </joint15_velocity_limit>
+    	<joint16_velocity_limit>1.0 </joint16_velocity_limit>
+    	<joint17_velocity_limit>1.0 </joint17_velocity_limit>
+    	<joint18_velocity_limit>1.0 </joint18_velocity_limit>
+    	<joint19_velocity_limit>1.0 </joint19_velocity_limit>
+    	<joint20_velocity_limit>1.0 </joint20_velocity_limit>
+    	<joint21_velocity_limit>1.0 </joint21_velocity_limit>
+    	<joint22_velocity_limit>1.0 </joint22_velocity_limit>
+    	<joint23_velocity_limit>1.0 </joint23_velocity_limit>
     </plugin>
   </gazebo>
+  <!-- Kinect v2 -->
+ <xacro:include filename="$(find kinect2_description)/urdf/kinect2/kinect2.xacro"/>
+ <kinect2_sensor parent="panda_arm_link8" prefix="" name="panda_arm_link8/kinect2" cam_px="0.0" cam_py="0" cam_pz="-0.20" cam_or="0" cam_op="0.52" cam_oy="0"/>
 </robot>
