Commit message: added a (urdf_models) ros package instead of using Gazebo models directory

File: ros_packages/src/franka_panda_arm_plus_allegro_right_hand_control_gazebo/model/franka_panda_arm_plus_allegro_right_hand_control_gazebo_plugin.urdf.xacro (robot description, xacro)
@@ -1,8 +1,14 @@
 <?xml version='1.0' encoding='utf-8'?>
 <robot xmlns:xacro="http://www.ros.org/wiki/xacro" name="panda_arm_plus_allegro_right_hand">
+  <xacro:property name="cell_name" value="master_cell" />
+  <!-- for .dae files visualization problem in Gazebo8 -->
+  <transparent opaque="RGB_ZERO"> <color>1 1 1 1</color> </transparent> <transparency><float>1</float></transparency>
+  <!-- Workcell frame model -->
+  <xacro:include filename="$(find urdf_models)/models/workcell_frame/workcell_frame.xacro"/>
+  <xacro:workcell_frame connected_to="" ns="${cell_name}" xyz="0 0 0.07" rpy="0 0 0" />
+  <!-- Franka-Panda arm model -->
   <xacro:include filename="$(find franka_panda_arm_description)/model/panda_arm_gazebo.xacro" />
-  <xacro:include filename="$(find allegro_right_hand_description)/model/allegro_right_hand.xacro"/>
-  <xacro:panda_arm arm_id="panda_arm" xyz="0.62 0.138 0.986" rpy="0 0 ${pi/2}" />
-  <transparent opaque="RGB_ZERO"> <color>1 1 1 1</color> </transparent> <transparency><float>1</float></transparency>
+  <xacro:panda_arm connected_to='${cell_name}_workcell_assembly' arm_id="panda_arm" xyz="0.62 0.138 0.986" rpy="0 0 ${pi/2}" />
+  <!-- Franka-Panda arm to Allegro hand connection -->
   <link name="franka_panda_arm_allegro_hand_connection">
     <visual>
@@ -30,6 +36,17 @@
     <origin xyz="0 0 0"/>
   </joint>
+  <!-- Allegro right hand model -->
+  <xacro:include filename="$(find allegro_right_hand_description)/model/allegro_right_hand.xacro"/>
   <!-- 0.0091=(-0.0113+0.0204) : -0.0113 to put the allegro hand Palm frame at zero position then add 0.0.0204(40.8mm/2) to put the same frame at center of panda-allegro-connection  -->
   <xacro:allegro_right_hand ns="panda_arm" x="-0.0091" y="0" z="0.02" roll="0" pitch="0" yaw="${pi}" connected_to="franka_panda_arm_allegro_hand_connection" />
+  <!-- ReadSense-d435 depth camera -->
+  <xacro:include filename="$(find realsense_d435_description)/model/realsense_d435.xacro"/>
+  <xacro:realsense_d435 connected_to="franka_panda_arm_allegro_hand_connection" ns="panda_arm" origin_rpy="0 ${-pi/2} 0" origin_xyz="-0.07 0 0" />
+  <gazebo>
+    <plugin name="RealSenseCamRosPlugin" filename="libRealSenseCamRosPlugin.so"> </plugin>
+  </gazebo>
+  <!-- Kinect v2 depth camera -->
+  <xacro:include filename="$(find kinect2_description)/urdf/kinect2/kinect2.xacro"/>
+  <kinect2_sensor parent="${cell_name}_workcell_assembly" prefix="" name="kinect2" cam_px="0.0" cam_py="0" cam_pz="2.40" cam_or="0" cam_op="0.52" cam_oy="0"/>
   <gazebo>
     <plugin name="generic_interface_plugin" filename="libgeneric_interface_plugin.so">
@@ -82,6 +99,3 @@
     </plugin>
   </gazebo>
-  <!-- Kinect v2 -->
- <xacro:include filename="$(find kinect2_description)/urdf/kinect2/kinect2.xacro"/>
- <kinect2_sensor parent="panda_arm_link8" prefix="" name="panda_arm_link8/kinect2" cam_px="0.0" cam_py="0" cam_pz="-0.20" cam_or="0" cam_op="0.52" cam_oy="0"/>
 </robot>

File: ros_packages/src/realsense_d435_description/model/realsense_d435.urdf.xacro (robot description, xacro)
@@ -2,52 +2,7 @@
 <robot xmlns:xacro="http://www.ros.org/wiki/xacro" name="realsense_d435">
   <xacro:include filename="$(find realsense_d435_description)/model/realsense_d435.xacro"/>
-  <xacro:realsense_d435 connected_to="" ns="real_sense" origin_rpy="0 0 0" origin_xyz="0 0 0.1" />
+  <xacro:realsense_d435 connected_to="" ns="real_sense1" origin_rpy="0 0 0" origin_xyz="0 0 0.1" />
   <gazebo>
     <plugin name="RealSenseCamRosPlugin" filename="libRealSenseCamRosPlugin.so"> </plugin>
   </gazebo>
-  <!--
-  <gazebo>
-  <plugin name="camera_plugin" filename="libgazebo_ros_openni_kinect.so">
-    <baseline>0.2</baseline>
-    <alwaysOn>true</alwaysOn>
-    <updateRate>0.0</updateRate>
-    <cameraName>camera_ir</cameraName>
-    <imageTopicName>/camera/depth/image_raw</imageTopicName>
-    <cameraInfoTopicName>/camera/depth/camera_info</cameraInfoTopicName>
-    <depthImageTopicName>/camera/depth/image_raw</depthImageTopicName>
-    <depthImageInfoTopicName>/camera/depth/camera_info</depthImageInfoTopicName>
-    <pointCloudTopicName>/camera/depth/points</pointCloudTopicName>
-    <frameName>camera_link</frameName>
-    <pointCloudCutoff>0.05</pointCloudCutoff>
-    <distortionK1>0</distortionK1>
-    <distortionK2>0</distortionK2>
-    <distortionK3>0</distortionK3>
-    <distortionT1>0</distortionT1>
-    <distortionT2>0</distortionT2>
-    <CxPrime>0</CxPrime>
-    <Cx>0</Cx>
-    <Cy>0</Cy>
-    <focalLength>0</focalLength>
-    <hackBaseline>0</hackBaseline>
-  </plugin>
-  </gazebo>
-   -->
-  <!--
-  <gazebo>
-  <plugin name="camera_controller" filename="libgazebo_ros_camera.so">
-    <alwaysOn>true</alwaysOn>
-    <updateRate>0.0</updateRate>
-    <cameraName>rrbot/camera1</cameraName>
-    <imageTopicName>image_raw</imageTopicName>
-    <cameraInfoTopicName>camera_info</cameraInfoTopicName>
-    <frameName>camera_link</frameName>
-    <hackBaseline>0.07</hackBaseline>
-    <distortionK1>0.0</distortionK1>
-    <distortionK2>0.0</distortionK2>
-    <distortionK3>0.0</distortionK3>
-    <distortionT1>0.0</distortionT1>
-    <distortionT2>0.0</distortionT2>
-  </plugin>
-  </gazebo>
-   -->
 </robot>

File: ros_packages/src/realsense_d435_description/model/realsense_d435.xacro (robot description, xacro)
@@ -134,6 +134,6 @@
         <horizontal_fov>0.7417</horizontal_fov>
         <image>
-          <width>1920</width>
-          <height>1080</height>
+          <width>640</width>
+          <height>480</height>
           <format>RGB_INT8</format>
         </image>
@@ -157,6 +157,6 @@
         <horizontal_fov>1.59174</horizontal_fov>
         <image>
-          <width>1280</width>
-          <height>800</height>
+          <width>640</width>
+          <height>480</height>
           <format>L_INT8</format>
         </image>
@@ -180,6 +180,6 @@
         <horizontal_fov>1.59174</horizontal_fov>
         <image>
-          <width>1280</width>
-          <height>800</height>
+          <width>640</width>
+          <height>480</height>
           <format>L_INT8</format>
         </image>

Commit message: more than one panda arm in simulation is possible now.

File: ros_packages/src/franka_panda_arm_plus_allegro_right_hand_control_gazebo/model/franka_panda_arm_plus_allegro_right_hand_control_gazebo_plugin.urdf.xacro (robot description, xacro)
@@ -1,5 +1,7 @@
 <?xml version='1.0' encoding='utf-8'?>
-<robot xmlns:xacro="http://www.ros.org/wiki/xacro" name="panda_arm_plus_allegro_right_hand">
+<robot xmlns:xacro="http://www.ros.org/wiki/xacro" name="master_cell">
   <xacro:property name="cell_name" value="master_cell" />
+  <xacro:property name="robot_arm1" value="panda1" />
+  <xacro:property name="robot_arm2" value="panda2" />
   <!-- for .dae files visualization problem in Gazebo8 -->
   <transparent opaque="RGB_ZERO"> <color>1 1 1 1</color> </transparent> <transparency><float>1</float></transparency>
@@ -9,38 +11,18 @@
   <!-- Franka-Panda arm model -->
   <xacro:include filename="$(find franka_panda_arm_description)/model/panda_arm_gazebo.xacro" />
-  <xacro:panda_arm connected_to='${cell_name}_workcell_assembly' arm_id="panda_arm" xyz="0.62 0.138 0.986" rpy="0 0 ${pi/2}" />
+  <xacro:panda_arm connected_to='${cell_name}_workcell_assembly' arm_id="${robot_arm1}" xyz="1.42 0.188 0.916" rpy="0 0 ${pi/2}" />
+  <xacro:panda_arm connected_to='${cell_name}_workcell_assembly' arm_id="${robot_arm2}" xyz="0.62 0.188 0.916" rpy="0 0 ${pi/2}" />
   <!-- Franka-Panda arm to Allegro hand connection -->
-  <link name="franka_panda_arm_allegro_hand_connection">
-    <visual>
-      <geometry>
-        <mesh filename="package://franka_panda_arm_plus_allegro_right_hand_control_gazebo/model/meshes/panda-allegro-connection.stl"/>
-      </geometry>
-      <origin rpy="0 0 ${pi/2}" xyz="0 0 0"/>
-    </visual>
-    <collision>
-      <geometry>
-        <mesh filename="package://franka_panda_arm_plus_allegro_right_hand_control_gazebo/model/meshes/panda-allegro-connection.stl"/>
-      </geometry>
-      <origin rpy="0 0 0" xyz="0 0 0"/>
-    </collision>
-    <inertial>
-      <origin xyz="0 0 0" rpy="0 0 0"/>
-      <mass value="0.1"/>
-      <inertia ixx="0.001" ixy="0.001" ixz="0.001" iyy="0.001" iyz="0.001" izz="0.001"/>
-    </inertial>
-  </link>
-  <gazebo reference="franka_panda_arm_allegro_hand_connection"><material>Gazebo/BlueGlow</material></gazebo>
-	<joint name="franka_panda_arm_allegro_hand_connection_joint" type="fixed">
-    <parent link="panda_arm_link8"/>
-    <child link="franka_panda_arm_allegro_hand_connection"/>
-    <origin xyz="0 0 0"/>
-  </joint>
+  <xacro:include filename="$(find urdf_models)/models/panda_allegro_connection/panda_allegro_connection.xacro"/>
+  <xacro:panda_allegro_connection connected_to="${robot_arm1}_link7" ns="${robot_arm1}" xyz="0 0 0.107" rpy="0 0 0" />
+  <xacro:panda_allegro_connection connected_to="${robot_arm2}_link7" ns="${robot_arm2}" xyz="0 0 0.107" rpy="0 0 0" />
   <!-- Allegro right hand model -->
   <xacro:include filename="$(find allegro_right_hand_description)/model/allegro_right_hand.xacro"/>
   <!-- 0.0091=(-0.0113+0.0204) : -0.0113 to put the allegro hand Palm frame at zero position then add 0.0.0204(40.8mm/2) to put the same frame at center of panda-allegro-connection  -->
-  <xacro:allegro_right_hand ns="panda_arm" x="-0.0091" y="0" z="0.02" roll="0" pitch="0" yaw="${pi}" connected_to="franka_panda_arm_allegro_hand_connection" />
+  <xacro:allegro_right_hand ns="${robot_arm1}" x="-0.0091" y="0" z="0.02" roll="0" pitch="0" yaw="${pi}" connected_to="${robot_arm1}_panda_allegro_connection" />
   <!-- ReadSense-d435 depth camera -->
   <xacro:include filename="$(find realsense_d435_description)/model/realsense_d435.xacro"/>
-  <xacro:realsense_d435 connected_to="franka_panda_arm_allegro_hand_connection" ns="panda_arm" origin_rpy="0 ${-pi/2} 0" origin_xyz="-0.07 0 0" />
+  <xacro:realsense_d435 connected_to="${robot_arm1}_panda_allegro_connection" ns="${robot_arm1}" origin_rpy="0 ${-pi/2} 0" origin_xyz="-0.0673 0 -0.02" />
+  <xacro:realsense_d435 connected_to="${robot_arm2}_panda_allegro_connection" ns="${robot_arm2}" origin_rpy="0 ${-pi/2} 0" origin_xyz="-0.0673 0 -0.02" />
   <gazebo>
     <plugin name="RealSenseCamRosPlugin" filename="libRealSenseCamRosPlugin.so"> </plugin>
@@ -48,5 +30,5 @@
   <!-- Kinect v2 depth camera -->
   <xacro:include filename="$(find kinect2_description)/urdf/kinect2/kinect2.xacro"/>
-  <kinect2_sensor parent="${cell_name}_workcell_assembly" prefix="" name="kinect2" cam_px="0.0" cam_py="0" cam_pz="2.40" cam_or="0" cam_op="0.52" cam_oy="0"/>
+  <kinect2_sensor parent="${cell_name}_workcell_assembly" prefix="" name="kinect2" cam_px="1.53" cam_py="0.567" cam_pz="2.188" cam_or="${pi/2}" cam_op="${pi/2}" cam_oy="0"/>
   <gazebo>
     <plugin name="generic_interface_plugin" filename="libgeneric_interface_plugin.so">
@@ -56,5 +38,5 @@
     	<joint4_init> -1.57</joint4_init>
     	<joint5_init> 0.00 </joint5_init>
-    	<joint6_init> 1.57</joint6_init>
+    	<joint6_init> 1.57 </joint6_init>
     	<joint7_init> 0.70 </joint7_init>
     	<joint8_init> 0.000</joint8_init>
@@ -74,4 +56,11 @@
     	<joint22_init>0.70 </joint22_init>
     	<joint23_init>0.30 </joint23_init>
+    	<joint24_init>0.00 </joint24_init>
+    	<joint25_init>-1.57</joint25_init>
+    	<joint26_init>0.00 </joint26_init>
+    	<joint27_init>-1.57</joint27_init>
+    	<joint28_init>0.00 </joint28_init>
+    	<joint29_init>1.57 </joint29_init>
+    	<joint30_init>0.70 </joint30_init>
     	<joint1_velocity_limit>1.0 </joint1_velocity_limit>
     	<joint2_velocity_limit>1.0 </joint2_velocity_limit>

File: ros_packages/src/realsense_d435_description/model/realsense_d435.xacro (robot description, xacro)
@@ -29,10 +29,10 @@
     <kinematic>0</kinematic>
     <gravity>1</gravity>
-    <visual name="visual">
+    <visual>
       <geometry>
         <mesh filename="package://${description_pkg}/model/meshes/d435.stl"/>
       </geometry>
     </visual>
-    <collision name='collision'>
+    <collision>
       <laser_retro>0</laser_retro>
       <max_contacts>10</max_contacts>
@@ -88,29 +88,29 @@
   </link>
   <!-- Virtual links representing the cameras positons and orientations-->
-  <link name="color" />
-  <link name="depth" />
-  <link name="stereo_right_imager" />
-  <link name="stereo_left_imager" />
+  <link name="${ns}_color" />
+  <link name="${ns}_depth" />
+  <link name="${ns}_stereo_right_imager" />
+  <link name="${ns}_stereo_left_imager" />
   <!-- Joints positioning the virtual links with respect to the camera main link-->
-  <joint name="color_joint" type="fixed">
-    <parent link="${ns}_link" />
-    <child link="color" />
+  <joint name="${ns}_color_joint" type="fixed">
+    <parent link="${ns}_link" />
+    <child link="${ns}_color" />
     <origin xyz="0 -0.0115 0" rpy="0 0 0"/>
     <!-- The default position is change since in Rviz the cloud depth axis is Z not X-->
     <!-- <origin xyz="0 -0.046 0.004" rpy="${pi/2} ${pi} ${pi/2}"/> -->
   </joint>
-  <joint name="stereo_right_imager_joint" type="fixed">
-    <parent link="${ns}_link" />
-    <child link="stereo_right_imager" />
+  <joint name="${ns}_stereo_right_imager_joint" type="fixed">
+    <parent link="${ns}_link" />
+    <child link="${ns}_stereo_right_imager" />
     <origin xyz="0 -0.0325 0" rpy="0 0 0"/>
   </joint>
-  <joint name="stereo_left_imager_joint" type="fixed">
-    <parent link="${ns}_link" />
-    <child link="stereo_left_imager" />
+  <joint name="${ns}_stereo_left_imager_joint" type="fixed">
+    <parent link="${ns}_link" />
+    <child link="${ns}_stereo_left_imager" />
     <origin xyz="0 0.0175 0" rpy="0 0 0"/>
   </joint>
-  <joint name="depth_joint" type="fixed">
-    <parent link="${ns}_link" />
-    <child link="depth" />
+  <joint name="${ns}_depth_joint" type="fixed">
+    <parent link="${ns}_link" />
+    <child link="${ns}_depth" />
     <origin xyz="0 -0.0115 0" rpy="0 0 0"/>
   </joint>
@@ -129,8 +129,9 @@
     <!--<max_vel>0.01</max_vel>
     <min_depth>0</min_depth>-->
-    <sensor name="color" type="camera">
+    <sensor name="${ns}_realsense_color" type="camera">
       <pose frame="">0 -0.0115 0 0 0 0</pose>
       <camera name="__default__">
-        <horizontal_fov>0.7417</horizontal_fov>
+        <!-- <horizontal_fov>0.7</horizontal_fov> -->
+        <horizontal_fov>1.27</horizontal_fov> <!-- 73 degrees -->
         <image>
           <width>640</width>
@@ -149,11 +150,12 @@
       </camera>
       <always_on>1</always_on>
-      <update_rate>60</update_rate>
+      <update_rate>30</update_rate>
       <visualize>1</visualize>
     </sensor>
-    <sensor name="stereo_right_imager" type="camera">
+    <sensor name="${ns}_realsense_stereo_right_imager" type="camera">
       <pose frame="">0 -0.0325 0 0 0 0</pose>
       <camera name="__default__">
-        <horizontal_fov>1.59174</horizontal_fov>
+        <!-- <horizontal_fov>1.59174</horizontal_fov> -->
+        <horizontal_fov>1.8</horizontal_fov> <!-- 103 degrees -->
         <image>
           <width>640</width>
@@ -172,11 +174,12 @@
       </camera>
       <always_on>1</always_on>
-      <update_rate>60</update_rate>
+      <update_rate>30</update_rate>
       <visualize>0</visualize>
     </sensor>
-    <sensor name="stereo_left_imager" type="camera">
+    <sensor name="${ns}_realsense_stereo_left_imager" type="camera">
       <pose frame="">0 0.0175 0 0 0 0</pose>
       <camera name="__default__">
-        <horizontal_fov>1.59174</horizontal_fov>
+        <!-- <horizontal_fov>1.59174</horizontal_fov> -->
+        <horizontal_fov>1.8</horizontal_fov> <!-- 103 degrees -->
         <image>
           <width>640</width>
@@ -195,27 +198,28 @@
       </camera>
       <always_on>1</always_on>
-      <update_rate>60</update_rate>
+      <update_rate>30</update_rate>
       <visualize>0</visualize>
     </sensor>
-    <sensor name="depth" type="depth">
+    <sensor name="${ns}_realsense_depth" type="depth">
       <pose frame="">0 -0.0115 0 0 0 0</pose>
       <camera name="__default__">
-        <horizontal_fov>1.047</horizontal_fov>
-        <image>
-          <width>640</width>
-          <height>480</height>
-        </image>
-        <clip>
-          <near>0.1</near>
-          <far>100</far>
-        </clip>
-        <noise>
-          <type>gaussian</type>
-          <mean>0.0</mean>
-          <stddev>0.007</stddev>
-        </noise>
-      </camera>
-      <always_on>1</always_on>
-      <update_rate>60</update_rate>
+        <!-- <horizontal_fov>1.047</horizontal_fov> -->
+        <horizontal_fov>1.623</horizontal_fov> <!-- 93 degrees -->
+        <image>
+          <width>640</width>
+          <height>480</height>
+        </image>
+        <clip>
+          <near>0.1</near>
+          <far>100</far>
+        </clip>
+        <noise>
+          <type>gaussian</type>
+          <mean>0.0</mean>
+          <stddev>0.007</stddev>
+        </noise>
+      </camera>
+      <always_on>1</always_on>
+      <update_rate>30</update_rate>
       <visualize>0</visualize>
     </sensor>
