Commit message: started torque control of arm + hand

File: ros_packages/src/franka_panda_arm_plus_allegro_right_hand_control_gazebo/model/workcell_one_robot_world_based.urdf.xacro (robot description, xacro)
@@ -6,12 +6,13 @@
   <transparent opaque="RGB_ZERO"> <color>1 1 1 1</color> </transparent> <transparency><float>1</float></transparency>
   <!-- Workcell frame model -->
-  <xacro:include filename="$(find urdf_models)/models/workcell_frame/workcell_frame.xacro"/>
-  <xacro:workcell_frame connected_to="" ns="${cell_name}" xyz="0 0 0.07" rpy="0 0 0" />
+  <!-- <xacro:include filename="$(find urdf_models)/models/workcell_frame/workcell_frame.xacro"/> -->
+  <!-- <xacro:workcell_frame connected_to="" ns="${cell_name}" xyz="0 0 0.07" rpy="0 0 0" /> -->
   <!-- Object model -->
-  <xacro:include filename="$(find urdf_models)/models/objects/cocacola_bottle.xacro"/>
-  <xacro:cocacola_bottle connected_to="" ns="" xyz="0.62 0.538 0.98" rpy="0 0 0" />
+  <!-- <xacro:include filename="$(find urdf_models)/models/objects/cocacola_bottle.xacro"/> -->
+  <!-- <xacro:cocacola_bottle connected_to='${cell_name}_workcell_assembly' ns="" xyz="1.2 0.6 0.91" rpy="0 0 0" /> -->
   <!-- Franka-Panda arm model -->
   <xacro:include filename="$(find franka_panda_arm_description)/model/panda_arm_gazebo.xacro" />
-  <xacro:panda_arm connected_to='${cell_name}_workcell_assembly' arm_id="${robot_arm1}" xyz="1.42 0.188 0.916" rpy="0 0 ${pi/2}" />
+  <!-- <xacro:panda_arm connected_to='${cell_name}_workcell_assembly' arm_id="${robot_arm1}" xyz="1.42 0.188 0.916" rpy="0 0 ${pi/2}" /> -->
+  <xacro:panda_arm connected_to="" arm_id="${robot_arm1}" xyz="1.42 0.188 0.916" rpy="0 0 ${pi/2}" />
   <!-- Franka-Panda arm to Allegro hand connection -->
   <xacro:include filename="$(find urdf_models)/models/panda_allegro_connection/panda_allegro_connection.xacro"/>

File: ros_packages/src/urdf_models/models/objects/cocacola_bottle.xacro (robot description, xacro)
@@ -11,7 +11,6 @@
   <!-- Used for fixing robot to Gazebo ground in case the robot is not connected to any other component -->
   <xacro:if value="${connected_to == ''}">
-	  <link name="world"/>
-	  <joint name="fix_to_world" type="continuous">
-		  <parent link="world"/>
+	  <joint name="fix_cocacola_bottle_to_world" type="continuous">
+		  <parent link="world"/>		<!-- here we assume the link "world" already exist in the tree -->
 		  <child link="cocacola_bottle"/>
 		  <origin xyz="${xyz}" rpy="${rpy}"/>
