Commit message: started using PCL

File: ros_packages/src/kinect2/model/kinect2.urdf.xacro (robot description, xacro)
@@ -1,8 +1,8 @@
 <?xml version="1.0"?>
 <robot xmlns:xacro="http://www.ros.org/wiki/xacro" name="kinect2_sensor">
-  <!-- <xacro:include filename="$(find kinect2_description)/model/kinect2.xacro" />
-  <xacro:kinect2_sensor ns="kinect" connected_to="" origin_xyz="0 0 0.5" origin_rpy="0 0 0" /> -->
+  <xacro:include filename="$(find kinect2)/model/kinect2.xacro" />
+  <xacro:kinect2_sensor ns="kinect" connected_to="" origin_xyz="0 0 0.5" origin_rpy="0 0 0" />
   <!-- Kinect v2 -->
- <xacro:include filename="$(find kinect2_description)/urdf/kinect2/kinect2.xacro"/>
- <kinect2_sensor parent="base_sensors" prefix="" name="kinect2" cam_px="0.0" cam_py="0" cam_pz="-0.20" cam_or="0" cam_op="0.52" cam_oy="0"/>
+ <!-- <xacro:include filename="$(find kinect2_description)/urdf/kinect2/kinect2.xacro"/>
+ <kinect2_sensor parent="base_sensors" prefix="" name="kinect2" cam_px="0.0" cam_py="0" cam_pz="-0.20" cam_or="0" cam_op="0.52" cam_oy="0"/> -->
 </robot>

File: ros_packages/src/kinect2/model/kinect2.xacro (robot description, xacro)
@@ -1,8 +1,5 @@
 <?xml version="1.0"?>
-<!-- This is a hand-made URDF XACRO file for the Microsoft Kinect-2 sensor (Xbox ONE) -->
-<!-- Copyright Universitaet Bremen - Instititute for Artificial Intelligence. Author: Alexis Maldonado -->
-<!-- License: GPLv3+ -->
 <robot xmlns:xacro="http://www.ros.org/wiki/xacro" name="kinect2_sensor">
-<xacro:macro name="kinect2_sensor" params=" ns:='' description_pkg:='kinect2_description' connected_to:='' origin_xyz:='0 0 0' origin_rpy:='0 0 0' ">
+<xacro:macro name="kinect2_sensor" params=" ns:='' description_pkg:='kinect2' connected_to:='' origin_xyz:='0 0 0' origin_rpy:='0 0 0' ">
   <material name="Kinect2Grey">
     <color rgba="0.15 0.15 0.15 1.0"/>

File: ros_packages/src/realsense_d435_description/model/realsense_d435.xacro (robot description, xacro)
@@ -151,5 +151,5 @@
       <always_on>1</always_on>
       <update_rate>30</update_rate>
-      <visualize>1</visualize>
+      <visualize>0</visualize>
     </sensor>
     <sensor name="${ns}_realsense_stereo_right_imager" type="camera">

File: ros_packages/src/urdf_models/models/workcell_frame/workcell_frame.xacro (robot description, xacro)
@@ -2,5 +2,5 @@
 <robot xmlns:xacro="http://www.ros.org/wiki/xacro" name="workcell_frame">
 <xacro:macro name="workcell_frame" params="ns:='robot_cell' description_pkg:='urdf_models' connected_to:='' xyz:='0 0 0.07' rpy:='0 0 0'">
-<static>true</static>
+<!-- <static>true</static> -->
 <xacro:unless value="${connected_to == ''}">
 	<joint name="${ns}_joint_${connected_to}" type="fixed">
