Commit message: repo update

File: ros_packages/src/franka_panda_arm_description_moveit/model/panda_arm_gazebo_moveit.urdf.xacro (robot description, xacro)
@@ -4,9 +4,11 @@
 	<xacro:include filename="$(find franka_panda_arm_description_moveit)/model/panda_arm_gazebo_moveit.xacro" />
 	<!-- <xacro:include filename="$(find franka_panda_arm_description_moveit)/model/hand.xacro" /> -->
-	<xacro:include filename="$(find franka_panda_arm_description_moveit)/model/panda_gazebo_friction.xacro" />
-	<xacro:include filename="$(find franka_panda_arm_description_moveit)/model/panda_gazebo_transmission.xacro" />
-	<xacro:panda_arm_moveit arm_id="panda" xyz="0 0 0.1" rpy="0 0 ${-pi/2}" />
-  <xacro:hand ns="panda" rpy="0 0 ${-pi/4}" connected_to="panda_link8"/>
-	<xacro:panda_gazebo robot_name="$(arg robot_name)" />
-	<xacro:panda_transmission robot_name="$(arg robot_name)" hardware_interface="$(arg hardware_interface)" />
+	<!-- <xacro:include filename="$(find franka_panda_arm_description_moveit)/model/panda_gazebo_friction.xacro" /> -->
+	<!-- <xacro:include filename="$(find franka_panda_arm_description_moveit)/model/panda_gazebo_transmission.xacro" /> -->
+	<!-- <xacro:panda_arm_moveit_friction robot_name="$(arg robot_name)" /> -->
+  <xacro:panda_arm_moveit arm_id="panda" xyz="0 0 0.1" rpy="0 0 ${-pi/2}" />
+  <!-- <xacro:hand ns="panda" rpy="0 0 ${-pi/4}" connected_to="panda_link8"/> -->
+  <!-- <xacro:panda_arm_moveit_transmission robot_name="$(arg robot_name)" /> -->
+	<!-- <xacro:panda_gazebo robot_name="$(arg robot_name)" /> -->
+	<!-- <xacro:panda_transmission robot_name="$(arg robot_name)" hardware_interface="$(arg hardware_interface)" /> -->
 </robot>

File: ros_packages/src/franka_panda_arm_description_moveit/model/panda_arm_gazebo_moveit.xacro (robot description, xacro)
@@ -260,4 +260,101 @@
 	<axis xyz="0 0 0"/>
 </joint>
+<gazebo reference="${arm_id}_link0">
+	<material>Gazebo/White</material>
+  <mu1>0.61</mu1>
+  <mu2>0.61</mu2>
+</gazebo>
+<gazebo reference="${arm_id}_link1">
+  <material>Gazebo/White</material>
+  <mu1>0.2</mu1>
+  <mu2>0.2</mu2>
+</gazebo>
+<gazebo reference="${arm_id}_link2">
+  <material>Gazebo/White</material>
+  <mu1>0.2</mu1>
+  <mu2>0.2</mu2>
+</gazebo>
+<gazebo reference="${arm_id}_link3">
+  <material>Gazebo/White</material>
+  <mu1>0.2</mu1>
+  <mu2>0.2</mu2>
+</gazebo>
+<gazebo reference="${arm_id}_link4">
+  <material>Gazebo/White</material>
+  <mu1>0.2</mu1>
+  <mu2>0.2</mu2>
+</gazebo>
+<gazebo reference="${arm_id}_link5">
+  <material>Gazebo/White</material>
+  <mu1>0.2</mu1>
+  <mu2>0.2</mu2>
+</gazebo>
+<gazebo reference="${arm_id}_link6">
+  <material>Gazebo/White</material>
+  <mu1>0.2</mu1>
+  <mu2>0.2</mu2>
+</gazebo>
+<gazebo reference="${arm_id}_link7">
+  <material>Gazebo/White</material>
+  <mu1>0.2</mu1>
+  <mu2>0.2</mu2>
+</gazebo>
+<gazebo>
+	<plugin name="gazebo_ros_control" filename="libgazebo_ros_control.so">
+	 <!-- <robotNamespace>/${robot_name}</robotNamespace> -->
+	</plugin>
+</gazebo>
+<transmission name="${arm_id}_tran_1">
+	<type>transmission_interface/SimpleTransmission</type>
+	<joint name="${arm_id}_joint1">
+		<hardwareInterface>hardware_interface/EffortJointInterface</hardwareInterface>
+	</joint>
+	<actuator name="${arm_id}_motor_1">
+		<hardwareInterface>hardware_interface/EffortJointInterface</hardwareInterface>
+	<mechanicalReduction>1</mechanicalReduction>
+	</actuator>
+	<joint name="${arm_id}_joint2">
+		<hardwareInterface>hardware_interface/EffortJointInterface</hardwareInterface>
+	</joint>
+	<actuator name="${arm_id}_motor_2">
+		<hardwareInterface>hardware_interface/EffortJointInterface</hardwareInterface>
+	<mechanicalReduction>1</mechanicalReduction>
+	</actuator>
+	<joint name="${arm_id}_joint3">
+		<hardwareInterface>hardware_interface/EffortJointInterface</hardwareInterface>
+	</joint>
+	<actuator name="${arm_id}_motor_3">
+		<hardwareInterface>hardware_interface/EffortJointInterface</hardwareInterface>
+	<mechanicalReduction>1</mechanicalReduction>
+	</actuator>
+	<joint name="${arm_id}_joint4">
+		<hardwareInterface>hardware_interface/EffortJointInterface</hardwareInterface>
+	</joint>
+	<actuator name="${arm_id}_motor_4">
+		<hardwareInterface>hardware_interface/EffortJointInterface</hardwareInterface>
+	<mechanicalReduction>1</mechanicalReduction>
+	</actuator>
+	<joint name="${arm_id}_joint5">
+		<hardwareInterface>hardware_interface/EffortJointInterface</hardwareInterface>
+	</joint>
+	<actuator name="${arm_id}_motor_5">
+		<hardwareInterface>hardware_interface/EffortJointInterface</hardwareInterface>
+	<mechanicalReduction>1</mechanicalReduction>
+	</actuator>
+	<joint name="${arm_id}_joint6">
+		<hardwareInterface>hardware_interface/EffortJointInterface</hardwareInterface>
+	</joint>
+	<actuator name="${arm_id}_motor_6">
+		<hardwareInterface>hardware_interface/EffortJointInterface</hardwareInterface>
+	<mechanicalReduction>1</mechanicalReduction>
+	</actuator>
+	<joint name="${arm_id}_joint7">
+		<hardwareInterface>hardware_interface/EffortJointInterface</hardwareInterface>
+	</joint>
+	<actuator name="${arm_id}_motor_7">
+		<hardwareInterface>hardware_interface/EffortJointInterface</hardwareInterface>
+	<mechanicalReduction>1</mechanicalReduction>
+	</actuator>
+</transmission>
 </xacro:macro>
 </robot>

File: ros_packages/src/franka_panda_arm_description_moveit/model/panda_gazebo_friction.xacro (robot description, xacro)
@@ -1,4 +1,5 @@
 <?xml version='1.0' encoding='utf-8'?>
-<robot xmlns:xacro="http://www.ros.org/wiki/xacro" name="panda_arm_moveit">
+<robot xmlns:xacro="http://www.ros.org/wiki/xacro" name="panda_arm_moveit_friction">
+<xacro:macro name="panda_arm_moveit_friction" params="robot_name:='' ">
 <gazebo reference="${robot_name}_link0">
 	<material>Gazebo/White</material>
@@ -41,3 +42,4 @@
   <mu2>0.2</mu2>
 </gazebo>
+</xacro:macro>
 </robot>

File: ros_packages/src/franka_panda_arm_description_moveit/model/panda_gazebo_transmission.xacro (robot description, xacro)
@@ -1,3 +1,5 @@
 <?xml version='1.0' encoding='utf-8'?>
+<robot xmlns:xacro="http://www.ros.org/wiki/xacro" name="panda_arm_moveit_transmission">
+<xacro:macro name="panda_arm_moveit_transmission" params="robot_name:='' ">
 <gazebo>
 	<plugin name="gazebo_ros_control" filename="libgazebo_ros_control.so">
@@ -57,2 +59,4 @@
 	</actuator>
 </transmission>
+</xacro:macro>
+</robot>
